File: keyboard.kicad_sch (KiCad schematic)
At the start: 68 parts, among them J1 Conn_01x04_Socket, J3 Conn_01x02_Socket, SW1 SW_Push, SW10 SW_Push, SW11 SW_Push, SW12 SW_Push, SW13 SW_Push, SW14 SW_Push, SW15 SW_Push, SW16 SW_Push, SW17 SW_Push, SW18 SW_Push, SW19 SW_Push, SW2 SW_Push, SW20 SW_Push, SW21 SW_Push, SW22 SW_Push, SW23 SW_Push, SW24 SW_Push, SW25 SW_Push, SW26 SW_Push, SW27 SW_Push, SW28 SW_Push, SW3 SW_Push, SW4 SW_Push, SW401 SW_Push, SW402 SW_Push, SW5 SW_Push, SW6 SW_Push, SW7 SW_Push, SW8 SW_Push, SW9 SW_Push, U1 rp2040-zero

Commit message: フットプリント更新
Parts:
- SW401: footprint Button_Switch_Keyboard:SW_Cherry_MX_2.00u_Plate -> kbd:keyswitch_cherrymx_hotswap_2u
- SW402: footprint Button_Switch_Keyboard:SW_Cherry_MX_2.00u_Vertical_Plate -> kbd:keyswitch_cherrymx_hotswap_2u_vertical
Changed lines of the file:
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@@
 			)
 		)
-		(property "Footprint" "Button_Switch_Keyboard:SW_Cherry_MX_2.00u_Vertical_Plate"
+		(property "Footprint" "kbd:keyswitch_cherrymx_hotswap_2u_vertical"
 			(at 143.51 137.16 0)
 			(effects
@@
 			)
 		)
-		(property "Footprint" "Button_Switch_Keyboard:SW_Cherry_MX_2.00u_Plate"
+		(property "Footprint" "kbd:keyswitch_cherrymx_hotswap_2u"
 			(at 93.98 137.16 0)
 			(effects

Commit message: なんとなく形になったので一旦commit
Parts:
- removed J1: Conn_01x04_Socket, Connector_PinHeader_2.54mm:PinHeader_1x04_P2.54mm_Vertical, symbol Connector:Conn_01x04_Socket
- added J1: Conn_01x06_Socket, Connector_PinHeader_2.54mm:PinHeader_1x06_P2.54mm_Vertical, symbol Connector:Conn_01x06_Socket
- SW5: renamed from SW401; footprint kbd:keyswitch_cherrymx_hotswap_2u -> kbd:keyswitch_cherrymx_hotswap_1u
- renumbered D9 to D10, D10 to D11, D11 to D12, D12 to D13, D13 to D14, D14 to D15, D15 to D16, D16 to D17, D17 to D18, D18 to D19, D402 to D20, D19 to D21, D20 to D22, D21 to D23, D22 to D24, D23 to D25, D24 to D26, D25 to D27, D26 to D28, D27 to D29, D28 to D30, D401 to D5, D5 to D6, D6 to D7, D7 to D8, D8 to D9, SW9 to SW10, SW10 to SW11, SW11 to SW12, SW12 to SW13, SW13 to SW14, SW14 to SW15, SW15 to SW16, SW16 to SW17, SW17 to SW18, SW18 to SW19, SW402 to SW20, SW19 to SW21, SW20 to SW22, SW21 to SW23, SW22 to SW24, SW23 to SW25, SW24 to SW26, SW25 to SW27, SW26 to SW28, SW27 to SW29, SW28 to SW30, SW5 to SW6, SW6 to SW7, SW7 to SW8, SW8 to SW9
Connections:
- net at U1.1 (0): now also J1.1 (Pin_1)
- net at JC1.S, R5.2, U1.16 (15)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: now also J1.5 (Pin_5)
- net at U1.2 (1): now also J1.2 (Pin_2)
- net at JC1.T, JP1.1 (A), R1.1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: now also J1.6 (Pin_6)
- net at U1.3 (2): now also J1.3 (Pin_3)
- net at U1.4 (3): now also J1.4 (Pin_4)
Other:
- moved on the sheet: J3, JC1, JP1, R1, R2, R5, U1
